File: schematics/cpe/cpe.kicad_sch (KiCad schematic)
At the start: 39 parts

Commit message: update CPE schematic
Parts:
- added L5, L6, L7: ~, symbol peppercorn:LUT1
- added M10, M11: ~, symbol peppercorn:MUX2
- added M9: ~, symbol peppercorn:MUX2 (conceptual)
- added U26, U33, U34: ~, symbol peppercorn:XOR
- added U27, U31: ~, symbol peppercorn:XOR3
- added U28, U29: ~, symbol peppercorn:AND
- added U30, U32: ~, symbol peppercorn:OR
- M7: symbol peppercorn:MUX2 -> peppercorn:MUX2 (conceptual)
Connections:
- net CINY1: now also U31.
- net COMB2OUT: now also U26.; no longer L4.D0, M3.Y
- net C_ADDF2: now also U30.
- net IN5: now also U28.
- net IN8: now also U29.
- net L02: now also M9.D0
- net L10: now also U27.
- net L11: now also M9.S, U31.
- net MUXOUT: now reaches M8.Y
- net TODO: FROM CLK: no longer names the net of U15.A
- net TODO: FROM CLK: now also L7.Y
- net TODO: FROM EN: no longer names the net of U17.A
- net TODO: FROM EN: now also L6.Y
- net TODO: FROM SR: no longer names the net of U18.A
- net TODO: FROM SR: now also L5.Y
- new net: L4.D0, M3.Y, U26.
- new net: U13., U5.
- new net: M10.D0, U27., U28.
- new net: M10.D1, M11.D1, U29., U31.
- new net: M11.S, U31., U32., U34.
- new net: M11.Y, U33.
- new net: M10.S, U27., U32., U33.
- new net: M9.Y, U30.
- new net "C": U26., U27., U30.
- new net CIN: C1.Y, M9.D1, U1., U13.
- new net CINY2: M11.D0, U34.
- new net CLK: L7.D
- new net COY2_S: U32.
- new net COY2_a: M10.Y
- new net EN: L6.D
- new net MULTO1: U34.
- new net MULTO2: U33.
- new net PINY2: U28., U29.
- new net SR: L5.D
Other:
- note added: "A[-1]"
- note added: "A[0]"
- note added: "B[1]"
- note added: "CI[0]"
- note added: "CI[1]"
- note added: "C_CLK"
- note added: "C_EN"
- note added: "C_R"
- note added: "L10 = (A[1] & B[0]) ^ SI[1] L11 = (A[0] & B[0]) ^ SI[0]"

Commit message: another CPE schematic update
Parts:
- removed U30: ~, symbol peppercorn:OR
- added U30: ~, symbol peppercorn:AND
Connections:
- net C_ADDF2: now also U30.
- net at M9.Y: now also U30.
- removed net "C": U26., U27.
- new net: U13., U5.
- new net: M10.D0, U27., U28.
- new net: M11.S, U31., U32., U34.
- new net: M10.S, U27., U32., U33.
- new net: U26., U27., U30.
Other:
- note added: "C_FUNCTION= 0: (none) 1; "C_ADDF": C_ADDF, C_ADDCIN 2; "C_ADDF2": C_ADDF, C_ADDF2, C_ADDCIN 3; "C_MULT": C_MULT, C_ADDF, C_ADDF2, C_ADDCIN 4; "C_MX4": C_MX4 5; "C_EN_CIN": C_EN_CIN 6; "C_CONCAT": C_ADDF 7; "C_ADDCIN": C_ADDCIN"
- note added: "In multiplier mode, the LUTs should be set up as: L10 = (A[1] & B[0]) ^ SI[1] L11 = (A[0] & B[0]) ^ SI[0]"
- note added: "This diagram is intended to be functionally correct, but when given a choice between ease of understanding and physical accuracy, I always chose the former. Dashed symbols represent where I'm describing something physically inaccurate. - Hannah Ravensloft"
- note removed: "A[-1]"
- note removed: "A[0]"
- note removed: "B[1]"
- note removed: "CI[0]"
- note removed: "CI[1]"
- note removed: "C_FUNCTION= 0: (none) 1: C_ADDF, C_ADDCIN 2: C_ADDF, C_ADDF2, C_ADDCIN 3: C_MULT, C_ADDF, C_ADDF2, C_ADDCIN 4: C_MX4 5: C_EN_CIN 6: C_CONCAT: C_ADDF 7: C_ADDCIN"
- note removed: "L10 = (A[1] & B[0]) ^ SI[1] L11 = (A[0] & B[0]) ^ SI[0]"
- note removed: "This diagram is intended to be functionally correct but when given a choice between ease of understanding and physical accuracy, I always chose the former. Dashed symbols represent where I'm describing something physically inaccurate. - Hannah Ravensloft"
- title: (none) -> Cologne Processing Element
