File: schematics/cpe/cpe_comb_en_cin.kicad_sch (KiCad schematic)
At the start: 13 parts

Commit message: another CPE schematic update
Other:
- company: (none) -> YosysHQ
Changed lines of the file:
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@@
 	(generator "eeschema")
 	(generator_version "9.0")
-	(paper "A4")
+	(paper "A3")
+	(title_block
+		(company "YosysHQ")
+	)
 	(rectangle
 		(start 19.05 60.325)
