File: schematics/cpe/prjpeppercorn.kicad_sch (KiCad schematic)
At the start: 0 parts

Commit message: another CPE schematic update
Other:
- company: (none) -> YosysHQ
Changed lines of the file:
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@@
 	(generator "eeschema")
 	(generator_version "9.0")
-	(paper "A4")
+	(paper "A3")
+	(title_block
+		(company "YosysHQ")
+	)
 	(sheet
 		(at 31.75 26.035)
